File: pcb/pongPCB.kicad_pcb (KiCad board)
At the start: 2 copper layers, 62.2 x 80 mm, 28 parts, among them U1 MCP4922, U2 TL082, U3 levelshift, U4 levelshift, U5 TL082, U6 NE555

Commit message: worked with Jordan to implement Nucleo shield.
Parts:
- removed ENC1, ENC2: Rotary_Encoder_Switch, Connector_PinHeader_2.54mm:PinHeader_1x05_P2.54mm_Vertical
- added SW1: Rotary_Encoder_Switch, Connector_PinHeader_2.54mm:PinHeader_1x05_P2.54mm_Vertical, F.Cu at (130.8, 130.8)
- added SW2: Rotary_Encoder_Switch, Connector_PinHeader_2.54mm:PinHeader_1x05_P2.54mm_Vertical, F.Cu at (130.8, 110.5)
Connections:
- net DT1 renamed /DT1
- net PA5-D13 renamed Net-(CN10-Pad11)
- net PA7-MOSI renamed Net-(CN10-Pad15)
- net PB6-D10 renamed Net-(CN10-Pad17)
- net PWM_output_to_laser renamed Net-(U6-Pad3)
- net X_ILDA-inverted renamed Net-(J1-Pad2)
- net X_ILDA-normal renamed Net-(J1-Pad3)
- net Y_ILDA-inverted renamed Net-(J2-Pad2)
- net Y_ILDA-normal renamed Net-(J2-Pad3)
- net button1 renamed /BUTTON1

Commit message: finished pcb layout. Ready for review
Parts:
- removed JP1, JP2: Jumper_3_Open, Jumper:SolderJumper-3_P1.3mm_Open_Pad1.0x1.5mm
- removed SW1, SW2: Rotary_Encoder_Switch, Connector_PinHeader_2.54mm:PinHeader_1x05_P2.54mm_Vertical
- added CN10: Conn_02x19_Odd_Even, Connector_PinHeader_2.54mm:PinHeader_2x19_P2.54mm_Vertical, F.Cu at (168.7, 59.3)
- added CN7: Conn_02x19_Odd_Even, Connector_PinHeader_2.54mm:PinHeader_2x19_P2.54mm_Vertical, F.Cu at (107.8, 59.5)
- added G***: LOGO, pcb:VSlogo, F.Cu at (527.6, 44.8)
- added G***: LOGO, pcb:VSlogo, B.Cu at (139.4, 119.5)
- added J1: X_ILDA_OUT, Connector_PinHeader_2.54mm:PinHeader_1x03_P2.54mm_Vertical, F.Cu at (175.8, 114.7)
- added J2: Y_ILDA_OUT, Connector_PinHeader_2.54mm:PinHeader_1x03_P2.54mm_Vertical, F.Cu at (175.8, 127.7)
- added J3: Xprobe, Connector_PinHeader_2.54mm:PinHeader_1x01_P2.54mm_Vertical, F.Cu at (129.1, 96.2)
- added J4: PowerInput, Connector_PinHeader_2.54mm:PinHeader_1x04_P2.54mm_Vertical, F.Cu at (107.4, 120.8)
- added J6: Yprobe, Connector_PinHeader_2.54mm:PinHeader_1x01_P2.54mm_Vertical, F.Cu at (137.2, 96.4)
- added J7: LaserToggle, Connector_PinHeader_2.54mm:PinHeader_1x01_P2.54mm_Vertical, F.Cu at (159.9, 59.6)
- added Joy1: Conn_01x05_Male, Connector_JST:JST_XH_B05B-XH-AM_1x05_P2.50mm_Vertical, F.Cu at (101.8, 140.3)
- added Joy2: Conn_01x05_Male, Connector_JST:JST_XH_B05B-XH-AM_1x05_P2.50mm_Vertical, F.Cu at (118.8, 140.3)
- added Rotary1: Rotary_Encoder_Switch, Connector_JST:JST_XH_B05B-XH-AM_1x05_P2.50mm_Vertical, F.Cu at (101.8, 129.3)
- added Rotary2: Rotary_Encoder_Switch, Connector_JST:JST_XH_B05B-XH-AM_1x05_P2.50mm_Vertical, F.Cu at (118.8, 129.3)
- added U7: 4081, Package_DIP:DIP-14_W7.62mm, F.Cu at (143.9, 59.8)
- added U8: 4081, Package_DIP:DIP-14_W7.62mm, F.Cu at (144.2, 83.4)
- added X-J1: XJumper1, Connector_PinHeader_2.54mm:PinHeader_1x03_P2.54mm_Vertical, F.Cu at (167.8, 113.5)
- added X-J2: XJumper2, Connector_PinHeader_2.54mm:PinHeader_1x03_P2.54mm_Vertical, F.Cu at (170.3, 113.5)
- added Y-J1: YJumper1, Connector_PinHeader_2.54mm:PinHeader_1x03_P2.54mm_Vertical, F.Cu at (167.5, 125.8)
- added Y-J2: YJumper2, Connector_PinHeader_2.54mm:PinHeader_1x03_P2.54mm_Vertical, F.Cu at (170.0, 125.8)
- moved RV5 75.2 mm to (134.9, 58.7), turned to 270 degrees
- moved RV2 73.6 mm to (136.0, 144.1), turned to 90 degrees
- moved D1 62.6 mm to (137.8, 65.1), turned to 270 degrees
- moved RV3 59.2 mm to (148.0, 144.1), turned to 90 degrees
- moved D2 52.0 mm to (132.9, 72.9), turned to 90 degrees
- moved R1 49.9 mm to (136.6, 132.2), turned to 0 degrees
- moved RV1 47.6 mm to (160.0, 144.1), turned to 90 degrees
- moved R3 45.7 mm to (148.4, 133.3)
- moved R4 45.7 mm to (148.4, 128.2)
- moved R7 45.7 mm to (148.4, 121.9)
- moved U2 45.7 mm to (135.7, 119.4)
- moved R5 45.7 mm to (148.4, 116.8)
- moved RV4 37.7 mm to (172.0, 144.1), turned to 90 degrees
- moved U6 35.0 mm to (129.5, 78.7)
- moved R2 28.9 mm to (154.3, 113.8), turned to 0 degrees
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Connections:
- U1 pad 8: GND -> /LATCH
- U3 pad 4: CLK2 -> /CLK1
- U4 pad 2: DT2 -> /DT2
- U4 pad 4: CLK2 -> /CLK2
- U4 pad 5: button2 -> /BUTTON2
Routing:
- net GND: track 0.00 -> 342.1 mm, vias 0 -> 5
- net +5V: track 8.67 -> 246.0 mm
- net Net-(J2-Pad3): track 0.00 -> 186.0 mm, vias 0 -> 5
- net Net-(Rotary1-Pad3): track 0.00 -> 154.9 mm, vias 0 -> 7
- net Net-(J3-Pad1): track 6.88 -> 153.1 mm, vias 0 -> 7
- net Net-(R1-Pad2): track 4.98 -> 132.9 mm
- net /DT1: track 0.00 -> 122.3 mm, vias 0 -> 1
- net /LASER_TOGGLE: track 0.00 -> 115.8 mm, vias 0 -> 4
- net Net-(R6-Pad2): track 0.00 -> 111.9 mm, vias 0 -> 6
- net +12V: track 0.00 -> 104.6 mm, vias 0 -> 5
- net /JOY2BUTTON: track 0.00 -> 103.9 mm
- net Net-(CN10-Pad7): track 0.00 -> 99.0 mm, vias 0 -> 2
- net /BUTTON2: track 0.00 -> 98.6 mm
- net Net-(D1-Pad2): track 0.00 -> 97.4 mm, vias 0 -> 3
- net Net-(J6-Pad1): track 0.00 -> 95.3 mm, vias 0 -> 4
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Other:
- board outline removed
- board text added: "LaserGameSystem V1"

Commit message: added edge cuts
Parts:
- removed the G*** at (527.6, 44.8)
Other:
- board outline added: 82 x 91.2 mm
