File: pcb/pongPCB.kicad_pcb (KiCad board)
At the start: 2 copper layers, 82 x 91.2 mm, 43 parts, among them CN10 Conn_02x19_Odd_Even, CN7 Conn_02x19_Odd_Even, J1 X_ILDA_OUT, J2 Y_ILDA_OUT, J3 Xprobe, J4 PowerInput, J6 Yprobe, J7 LaserToggle, U1 MCP4922, U2 TL082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

Commit message: state of PCB at time of first order
Parts:
- U3, U4: footprint Package_DIP:DIP-12_W7.62mm -> Package_DIP:DIP-12_W10.16mm
- moved U3 0.99 mm to (114.0, 103.3)
- moved U4 0.50 mm to (114.7, 83.2)
Connections:
- CN10 pad 7: Net-(CN10-Pad7) -> +5V
- CN7 pad 16: Net-(CN10-Pad7) -> +3V3
- CN7 pad 18: Net-(CN7-Pad18) -> +5V
- U3 pad 1: +5V -> /DT1
- U3 pad 10: Net-(Rotary1-Pad1) -> +12V
- U3 pad 11: +12V -> Net-(U3-Pad11)
- U3 pad 12: Net-(U3-Pad12) -> Net-(Rotary1-Pad1)
- U3 pad 2: /DT1 -> Net-(U3-Pad2)
- U3 pad 3: Net-(U3-Pad3) -> +3V3
- U3 pad 4: /CLK1 -> GND
- U3 pad 5: /BUTTON1 -> /CLK1
- U3 pad 6: GND -> /BUTTON1
- U3 pad 9: Net-(U3-Pad9) -> GND
- U4 pad 1: +5V -> /DT2
- U4 pad 10: Net-(Rotary2-Pad1) -> +12V
- U4 pad 11: +12V -> Net-(U4-Pad11)
- U4 pad 12: Net-(U4-Pad12) -> Net-(Rotary2-Pad1)
- U4 pad 2: /DT2 -> Net-(U4-Pad2)
- U4 pad 3: Net-(U4-Pad3) -> +3V3
- U4 pad 4: /CLK2 -> GND
- U4 pad 5: /BUTTON2 -> /CLK2
- U4 pad 6: GND -> /BUTTON2
- U4 pad 9: Net-(U4-Pad9) -> GND
Routing:
- net +3V3: track 0.00 -> 101.0 mm, vias 0 -> 1
- net Net-(CN10-Pad7): track 99.0 -> 0.00 mm, vias 2 -> 0
- net GND: track 342.1 -> 385.4 mm, vias 5 -> 7
- net +5V: track 246.0 -> 280.5 mm, vias 0 -> 3
- net /DT1: track 122.3 -> 93.3 mm, vias 1 -> 0
- net -15V: track 79.9 -> 63.9 mm, vias 3 -> 5
- net Net-(Rotary2-Pad1): track 50.8 -> 63.8 mm, vias 0 -> 2
- net Net-(Rotary1-Pad5): track 36.8 -> 24.5 mm, vias 0 -> 1
- net Net-(Rotary2-Pad3): track 59.8 -> 47.8 mm
- net /BUTTON2: track 98.6 -> 90.9 mm
- net Net-(Rotary1-Pad1): track 37.5 -> 43.3 mm
- net Net-(Rotary1-Pad3): track 154.9 -> 150.4 mm
- net /CLK2: track 71.2 -> 73.9 mm, vias 1 -> 2
- net /DT2: track 70.0 -> 72.7 mm, vias 3 -> 4
- net /LASER_TOGGLE: track 115.8 -> 117.8 mm
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Other:
- outline, holes or cut-outs redrawn
